File: circuit/circuit.brd (EAGLE design)
At the start: 100 x 80 mm, 78 parts

Commit message: initial changes from elias
Parts:
- removed CD1, CD2: 100pF, rcl:C025-025X050
- removed CD3: 100nF, rcl:C025-025X050
- removed DD1, DD2: 1N4148, diode:DO35-7
- removed ICD: DRIVER_RS485, robo_ag:IC_DIL08
- removed ICL1, ICL2: ULN2003AN, uln-udn:DIL16
- removed J201, J202: (no value), robo_ag:STECKER_WANNE_10
- removed J301, J303: (no value), pinhead:1X03
- removed JD1, JD2, JD3, JD4: (no value), pinhead:1X02
- removed JLED1, JLED2: MICROMATCH-6, con-amp-micromatch:MICROMATCH-6
- removed JP6: (no value), pinhead:1X06/90
- removed LD1: red, robo_ag:LED_3MM
- removed LD2: green, robo_ag:LED_3MM
- removed LED3: LED_3X, robo_ag:LED_TOP_PLCC6
- removed RD1, RD6, RL1I, RL2I: 150, rcl:0207/10
- removed RD2: 100k, rcl:0207/10
- removed RD3, RD4: ?, rcl:0207/10
- removed RD5, RD7: 1k, rcl:0207/10
- removed RD8, RD9: 10k, rcl:0207/10
- removed RL1B, RL1G, RL2B, RL2G, RL3B, RL3G: 22, rcl:0207/10
- removed RL1R, RL2R, RL3R: 40,4, rcl:0207/10
- removed RLD1, RLD2: 2k, rcl:0207/10
- added CM4, CM5, CM6: 100nF, rcl:C025-025X050
- added H1, H2, H3, H4: MOUNT-HOLE3.2, holes:3,2
- added IC1, IC2, IC4: 74HC86N, 74xx-eu:DIL14
- added IC3: 74HC30N, 74xx-eu:DIL14
- added JP1: IN, pinhead:1X08
- added SJ1, SJ2, SJ3, SJ4, SJ5, SJ6, SJ7, SJ8: (no value), jumper:SJ
- added SV1, SV2: (no value), con-harting-ml:ML10
Connections:
- net BTNMODE renamed BTN3
- removed net BUS_A: DD1.A, ICD.6, J201.5, J202.5, JD1.2, RD6.2
- removed net BUS_B: DD2.A, ICD.7, J201.6, J202.6, JD2.2, RD7.2
- removed net BUS_DETECT1: CD1.1, ICM.12, JD4.2, RD1.2, RD2.2
- removed net BUS_DETECT2: CD2.1, ICM.13, RD3.2, RD4.2
- removed net BUS_ENABLE: ICD.3, ICM.4, RD9.1, RLD2.1
- removed net BUS_RX: ICD.1, ICM.2, RLD1.2
- removed net BUS_TX: ICD.4, ICM.3
- removed net IRLED1: ICL1.7, ICM.5
- removed net IRLED1_OUT: ICL1.10, RL1I.1
- removed net IRLED2_MOSI: ICL2.7, ICM.17, RP.2
- removed net IRLED2_OUT: ICL2.10, RL2I.1
- removed net LED1_B: ICL1.5, ICL1.6, ICM.11
- removed net LED1_B_OUT: ICL1.11, ICL1.12, RL1B.1, RL3B.1
- removed net LED1_G: ICL1.3, ICL1.4, ICM.16
- removed net LED1_G_OUT: ICL1.13, ICL1.14, RL1G.1, RL3G.1
- removed net LED1_R: ICL1.1, ICL1.2, ICM.15
- removed net LED1_R_OUT: ICL1.15, ICL1.16, RL1R.1, RL3R.1
- removed net LED2_B: ICL2.5, ICL2.6, ICM.25, JP6.2
- removed net LED2_B_OUT: ICL2.11, ICL2.12, RL2B.1
- removed net LED2_G: ICL2.3, ICL2.4, ICM.24, JP6.3
- removed net LED2_G_OUT: ICL2.13, ICL2.14, RL2G.1
- removed net LED2_R: ICL2.1, ICL2.2, ICM.23, JD4.1, JP6.4
- removed net LED2_R_OUT: ICL2.15, ICL2.16, RL2R.1
- removed net N$32: ICD.2, RD8.1
- removed net N$33: JD2.1, RD6.1
- removed net N$34: LD1.K, RLD1.1
- removed net N$35: JD3.1, RD7.1
- removed net N$36: DD1.C, DD2.C, RD1.1
- removed net N$37: LD2.A, RLD2.2
- new net BUS_BTN_DATA: IC2.1, SV1.8
- new net BUS_BTN_LOAD: IC1.12, SV1.7
- new net BUS_CLK: IC1.1, SV1.2
- new net BUS_ERROR: IC3.8
- new net BUS_IR_CLK: IC1.9, SV1.6
- new net BUS_LED_DATA: IC2.9, SV1.10
- new net BUS_LED_LOAD: IC2.4, SV1.9
- new net BUS_RGB: IC1.4, SV1.4
- new net DISP_!ENABLE!: JP1.8
- new net DISP_COL_SCK: JP1.6
- new net DISP_COL_SER: JP1.4
- new net DISP_RCK: JP1.7
- new net DISP_ROW_SCK: JP1.5
- new net DISP_ROW_SER: JP1.3
- new net N$1: IC3.1, SJ1.2
- new net N$2: IC3.2, SJ2.2
- new net N$3: IC3.3, SJ3.2
- new net PROG_MOSI: ICM.17, RP.2
- new net RETURN_BTN_DATA: IC2.2, SV2.8
- new net RETURN_BTN_LOAD: IC1.13, SV2.7
- new net RETURN_CLK: IC1.2, SV2.2
- new net RETURN_IR_CLK: IC1.10, SV2.6
- new net RETURN_LED_DATA: IC2.10, SV2.10
- new net RETURN_LED_LAOD: IC2.5
- new net RETURN_LED_LOAD: SV2.9
- new net RETURN_RGB: IC1.5, SV2.4
- new net VCC: IC3.14
- net +5V: now also CM4.2, CM5.2, CM6.2, IC1.14, IC2.14, IC4.14, JP1.2, SJ8.1; no longer CD3.1, ICD.8, ICL1.9, ICL2.9, J201.1, J201.10, J201.3, J201.8, J202.1, J202.10, J202.3, J202.8, J301.1, J301.3, J303.1, J303.3, JLED1.1, JLED1.3, JLED1.5, JLED2.1, JLED2.3, JLED2.5, JP6.5, LD1.A, LED3.1, LED3.3, LED3.4, RD3.1, RD5.2
- net BTN2: no longer JP6.1
- net GND: now also CM4.1, CM5.1, CM6.1, IC1.7, IC2.12, IC2.13, IC2.7, IC3.7, IC4.7, JP1.1, SV1.1, SV1.3, SV1.5, SV2.1, SV2.3, SV2.5; no longer CD1.2, CD2.2, CD3.2, ICD.5, ICL1.8, ICL2.8, J201.2, J201.4, J201.7, J201.9, J202.2, J202.4, J202.7, J202.9, JD3.2, JP6.6, LD2.K, RD2.1, RD4.1, RD8.2, RD9.2
- net N$16: now also IC3.4, SJ4.2; no longer JLED1.2, RL1R.2
- net N$17: now also IC3.5, SJ5.2; no longer JLED1.4, RL1G.2
- net N$18: now also IC3.6, SJ6.2; no longer JLED1.6, RL1B.2
- net N$19: now also IC3.11, SJ7.2; no longer JLED2.2, RL2R.2
- net N$20: now also IC3.12, SJ8.2; no longer JLED2.4, RL2G.2
- net N$21: now also IC1.3, SJ1.1; no longer JLED2.6, RL2B.2
- net N$22: now also IC1.6, SJ2.1; no longer J303.2, RL2I.2
- net N$23: now also IC1.8, SJ3.1; no longer J301.2, RL1I.2
- net N$24: now also IC1.11, SJ4.1; no longer LED3.6, RL3R.2
- net N$25: now also IC2.3, SJ5.1; no longer LED3.2, RL3G.2
- net N$26: now also IC2.6, SJ6.1; no longer LED3.5, RL3B.2
- net N$31: now also IC2.8, SJ7.1; no longer JD1.1, RD5.1
Routing:
- net GND: track 675.6 -> 439.4 mm, vias 11 -> 6
- net +5V: track 608.5 -> 448.4 mm, vias 7 -> 6
- net BUS_A: track 144.8 -> 0.00 mm, vias 2 -> 0
- net BUS_B: track 130.6 -> 0.00 mm, vias 1 -> 0
- net IRLED2_MOSI: track 85.8 -> 0.00 mm, vias 1 -> 0
- net LED2_R: track 74.4 -> 0.00 mm
- net LED2_G: track 65.3 -> 0.00 mm
- net LED2_B: track 62.0 -> 0.00 mm
- net BUS_RX: track 51.7 -> 0.00 mm, vias 1 -> 0
- net LED1_B_OUT: track 47.0 -> 0.00 mm
- net BUS_ENABLE: track 46.6 -> 0.00 mm
- net LED1_R_OUT: track 46.4 -> 0.00 mm
- net LED1_R: track 46.1 -> 0.00 mm
- net BUS_TX: track 42.1 -> 0.00 mm, vias 1 -> 0
- net BUS_DETECT1: track 41.1 -> 0.00 mm
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Other:
- board text removed: "10.01.17"
- board text removed: "B1"
- board text removed: "B2"
- board text removed: "BM"
- board text removed: "IR1"
- board text removed: "IR2"
- board text removed: "P. Weissig"
- board text removed: "PullDown"
- board text removed: "PullUp"
- board text removed: "PvP"
- board text removed: "R X"
- board text removed: "RGB1"
- board text removed: "RGB2"
- board text removed: "RoboSAX"
- board text removed: "T X"
- board text removed: "TWI"
- board text removed: "Term"
