File: circuit/circuit.sch (EAGLE design)
At the start: 78 parts

Commit message: initial changes from elias
Parts:
- removed CD1, CD2: 100pF, rcl:C-EU025-025X050
- removed CD3: 100nF, rcl:C-EU025-025X050
- removed DD1, DD2: 1N4148, diode:1N4148DO35-7
- removed ICD: DRIVER_RS485, robo_ag:DRIVER_RS485
- removed ICL1, ICL2: ULN2003AN, uln-udn:ULN2003AN
- removed J201, J202: (no value), robo_ag:STECKER_WANNE_10
- removed J301, J303: (no value), pinhead:PINHD-1X3
- removed JD1, JD2, JD3, JD4: (no value), pinhead:PINHD-1X2
- removed JLED1, JLED2: MICROMATCH-6, con-amp-micromatch:MICROMATCH-6
- removed JP6: (no value), pinhead:PINHD-1X6/90
- removed LD1: red, robo_ag:LED-3MM
- removed LD2: green, robo_ag:LED-3MM
- removed LED3: LED_3X, robo_ag:LED_3X
- removed RD1, RD6, RL1I, RL2I: 150, rcl:R-EU_0207/10
- removed RD2: 100k, rcl:R-EU_0207/10
- removed RD3, RD4: ?, rcl:R-EU_0207/10
- removed RD5, RD7: 1k, rcl:R-EU_0207/10
- removed RD8, RD9: 10k, rcl:R-EU_0207/10
- removed RL1B, RL1G, RL2B, RL2G, RL3B, RL3G: 22, rcl:R-EU_0207/10
- removed RL1R, RL2R, RL3R: 40,4, rcl:R-EU_0207/10
- removed RLD1, RLD2: 2k, rcl:R-EU_0207/10
- added CM4, CM5, CM6: 100nF, rcl:C-EU025-025X050
- added H1, H2, H3, H4: MOUNT-HOLE3.2, holes:MOUNT-HOLE3.2
- added IC1, IC2, IC4: 74HC86N, 74xx-eu:74HC86N
- added IC3: 74HC30N, 74xx-eu:74HC30N
- added JP1: IN, pinhead:PINHD-1X8
- added SJ1, SJ2, SJ3, SJ4, SJ5, SJ6, SJ7, SJ8: (no value), jumper:SJ
- added SV1, SV2: (no value), con-harting-ml:ML10
Connections:
- net BTNMODE renamed BTN3
- removed net BUS_A: DD1.A, ICD.A, J201.5, J202.5, JD1.2, RD6.2
- removed net BUS_B: DD2.A, ICD.B, J201.6, J202.6, JD2.2, RD7.2
- removed net BUS_DETECT1: CD1.1, ICM.PD6(AIN0), JD4.2, RD1.2, RD2.2
- removed net BUS_DETECT2: CD2.1, ICM.PD7(AIN1), RD3.2, RD4.2
- removed net BUS_ENABLE: ICD.DE, ICM.PD2(INT0), RD9.1, RLD2.1
- removed net BUS_RX: ICD.R, ICM.PD0(RXD), RLD1.2
- removed net BUS_TX: ICD.D, ICM.PD1(TXD)
- removed net IRLED1: ICL1.I7, ICM.PD3(INT1)
- removed net IRLED1_OUT: ICL1.O7, RL1I.1
- removed net IRLED2_MOSI: ICL2.I7, ICM.PB3(MOSI/OC2), RP.2
- removed net IRLED2_OUT: ICL2.O7, RL2I.1
- removed net LED1_B: ICL1.I5, ICL1.I6, ICM.PD5(T1)
- removed net LED1_B_OUT: ICL1.O5, ICL1.O6, RL1B.1, RL3B.1
- removed net LED1_G: ICL1.I3, ICL1.I4, ICM.PB2(SS/OC1B)
- removed net LED1_G_OUT: ICL1.O3, ICL1.O4, RL1G.1, RL3G.1
- removed net LED1_R: ICL1.I1, ICL1.I2, ICM.PB1(OC1A)
- removed net LED1_R_OUT: ICL1.O1, ICL1.O2, RL1R.1, RL3R.1
- removed net LED2_B: ICL2.I5, ICL2.I6, ICM.PC2(ADC2), JP6.2
- removed net LED2_B_OUT: ICL2.O5, ICL2.O6, RL2B.1
- removed net LED2_G: ICL2.I3, ICL2.I4, ICM.PC1(ADC1), JP6.3
- removed net LED2_G_OUT: ICL2.O3, ICL2.O4, RL2G.1
- removed net LED2_R: ICL2.I1, ICL2.I2, ICM.PC0(ADC0), JD4.1, JP6.4
- removed net LED2_R_OUT: ICL2.O1, ICL2.O2, RL2R.1
- removed net N$32: ICD.!RE, RD8.1
- removed net N$33: JD2.1, RD6.1
- removed net N$34: LD1.C, RLD1.1
- removed net N$35: JD3.1, RD7.1
- removed net N$36: DD1.C, DD2.C, RD1.1
- removed net N$37: LD2.A, RLD2.2
- new net BUS_BTN_DATA: IC2A.I0, SV1.8
- new net BUS_BTN_LOAD: IC1D.I0, SV1.7
- new net BUS_CLK: IC1A.I0, SV1.2
- new net BUS_ERROR: IC3A.O
- new net BUS_IR_CLK: IC1C.I0, SV1.6
- new net BUS_LED_DATA: IC2C.I0, SV1.10
- new net BUS_LED_LOAD: IC2B.I0, SV1.9
- new net BUS_RGB: IC1B.I0, SV1.4
- new net DISP_!ENABLE!: JP1.8
- new net DISP_COL_SCK: JP1.6
- new net DISP_COL_SER: JP1.4
- new net DISP_RCK: JP1.7
- new net DISP_ROW_SCK: JP1.5
- new net DISP_ROW_SER: JP1.3
- new net N$1: IC3A.I0, SJ1.2
- new net N$2: IC3A.I1, SJ2.2
- new net N$3: IC3A.I2, SJ3.2
- new net PROG_MOSI: ICM.PB3(MOSI/OC2), RP.2
- new net RETURN_BTN_DATA: IC2A.I1, SV2.8
- new net RETURN_BTN_LOAD: IC1D.I1, SV2.7
- new net RETURN_CLK: IC1A.I1, SV2.2
- new net RETURN_IR_CLK: IC1C.I1, SV2.6
- new net RETURN_LED_DATA: IC2C.I1, SV2.10
- new net RETURN_LED_LAOD: IC2B.I1
- new net RETURN_LED_LOAD: SV2.9
- new net RETURN_RGB: IC1B.I1, SV2.4
- net +5V: now also CM4.2, CM5.2, CM6.2, IC1P.VCC, IC2P.VCC, IC4P.VCC, JP1.2, SJ8.1; no longer CD3.1, ICD.VCC, ICL1.CD+, ICL2.CD+, J201.1, J201.10, J201.3, J201.8, J202.1, J202.10, J202.3, J202.8, J301.1, J301.3, J303.1, J303.3, JLED1-1.S, JLED1-3.S, JLED1-5.S, JLED2-1.S, JLED2-3.S, JLED2-5.S, JP6.5, LD1.A, LED3-B.A, LED3-G.A, LED3-R.A, RD3.1, RD5.2
- net BTN2: no longer JP6.1
- net GND: now also CM4.1, CM5.1, CM6.1, IC1P.GND, IC2D.I0, IC2D.I1, IC2P.GND, IC4P.GND, JP1.1, SV1.1, SV1.3, SV1.5, SV2.1, SV2.3, SV2.5; no longer CD1.2, CD2.2, CD3.2, ICD.GND, ICL1.GND, ICL2.GND, J201.2, J201.4, J201.7, J201.9, J202.2, J202.4, J202.7, J202.9, JD3.2, JP6.6, LD2.C, RD2.1, RD4.1, RD8.2, RD9.2
- net N$16: now also IC3A.I3, SJ4.2; no longer JLED1-2.S, RL1R.2
- net N$17: now also IC3A.I4, SJ5.2; no longer JLED1-4.S, RL1G.2
- net N$18: now also IC3A.I5, SJ6.2; no longer JLED1-6.S, RL1B.2
- net N$19: now also IC3A.I6, SJ7.2; no longer JLED2-2.S, RL2R.2
- net N$20: now also IC3A.I7, SJ8.2; no longer JLED2-4.S, RL2G.2
- net N$21: now also IC1A.O, SJ1.1; no longer JLED2-6.S, RL2B.2
- net N$22: now also IC1B.O, SJ2.1; no longer J303.2, RL2I.2
- net N$23: now also IC1C.O, SJ3.1; no longer J301.2, RL1I.2
- net N$24: now also IC1D.O, SJ4.1; no longer LED3-R.C, RL3R.2
- net N$25: now also IC2A.O, SJ5.1; no longer LED3-G.C, RL3G.2
- net N$26: now also IC2B.O, SJ6.1; no longer LED3-B.C, RL3B.2
- net N$31: now also IC2C.O, SJ7.1; no longer JD1.1, RD5.1
Other:
- note added: "Anzeige Connector"
- note added: "Nochmal drüber nachdenken! Über die Jumper können die gewünschten Signale gewählt werden. Allerdings müssen freie Eingänge mit VDD verbunden werden. Hier ist noch eine clevere Lösung nötig."
- note removed: "(!OE)"
- note removed: "(DS)"
- note removed: "(Shift)"
- note removed: "(Store)"
- note removed: "Data 1"
- note removed: "Data 2"
- note removed: "Data 3"
- note removed: "Data 4"
- note removed: "GND"
- note removed: "LED"
- note removed: "LED-Driver"
- note removed: "Note: Possible extended Bus-Detection through ADC-Pin 0. E.g. Idle-Detection. Only if in single-light-mode (not 2 lights). ==> Therefore using a jumper"
- note removed: "Note: SN75176 & ADM485 share the same layout."
- note removed: "Note: Using atmega8 schematics. Pin-layout is the same."
- note removed: "Note: Value of RD3 and RD4 depend on ICD! SN75176: RD3= ; RD4= ADM485: RD3= ; RD4="
- note removed: "Vcc"
- moved on the sheet: J501-1, J501-2, J502-1, J502-2
